File: hardware/OsmoIRSensor.sch (KiCad schematic (older format))
At the start: 11 parts, among them J2 CONN_02X03_PCB_DIRECT, U1 ATTINY45-S, U2 TSOP75436WTR, X1 20MHz

Commit message: - Corrected IC Pads Size - Gerber Files added for 10x9,1cm panelized pcb - 3D Printer Files for optical Barrier added - Pin Desc. for DEV Cabel
Other:
- note added: "J2 Stecker\n1. VCC GRAU 2\n2. MOSI GELB 6\n3. GND GRUEN 5\n4. MISO WEISS 1\n5. SCK ROSA 3\n6. RESET BRAU 4"
Changed lines of the file:
@@
 Text Notes 1900 1175 0    60   ~ 0
 The IR-DEV Version connects all Pins of J2 to the outside. That makes it possible to reprogramm or analyze the ATTINY or signals. The consumer version just needs 3 pins connected to the outside\n\nPIN1 +5V\nPIN3 GND\nPIN5 SensorOut
+Text Notes 7450 1625 0    60   ~ 12
+J2                     Stecker\n1. VCC GRAU       2\n2. MOSI GELB       6\n3. GND GRUEN     5\n4. MISO WEISS      1\n5. SCK ROSA         3\n6. RESET BRAU     4
 $EndSCHEMATC
